Commit message: Updated URDF file

File: robot_quadruped/src/robot_description/urdf/robot.urdf (robot description, URDF)
Before this commit: robot robot, 13 links, 12 joints
Joints:
- joint Revolution 1: limit (none) -> lower=-1.57 upper=1.57 effort=10.0 velocity=5.0; type continuous -> revolute
- joint Revolution 10: limit (none) -> lower=-1.57 upper=1.57 effort=10.0 velocity=5.0; type continuous -> revolute
- joint Revolution 11: limit (none) -> lower=-1.57 upper=1.57 effort=10.0 velocity=5.0; type continuous -> revolute
- joint Revolution 12: limit (none) -> lower=-1.57 upper=1.57 effort=10.0 velocity=5.0; type continuous -> revolute
- joint Revolution 2: limit (none) -> lower=-1.57 upper=1.57 effort=10.0 velocity=5.0; type continuous -> revolute
- joint Revolution 3: limit (none) -> lower=-1.57 upper=1.57 effort=10.0 velocity=5.0; type continuous -> revolute
- joint Revolution 4: limit (none) -> lower=-1.57 upper=1.57 effort=10.0 velocity=5.0; type continuous -> revolute
- joint Revolution 5: limit (none) -> lower=-1.57 upper=1.57 effort=10.0 velocity=5.0; type continuous -> revolute
- joint Revolution 6: limit (none) -> lower=-1.57 upper=1.57 effort=10.0 velocity=5.0; type continuous -> revolute
- joint Revolution 7: limit (none) -> lower=-1.57 upper=1.57 effort=10.0 velocity=5.0; type continuous -> revolute
- joint Revolution 8: limit (none) -> lower=-1.57 upper=1.57 effort=10.0 velocity=5.0; type continuous -> revolute
- joint Revolution 9: limit (none) -> lower=-1.57 upper=1.57 effort=10.0 velocity=5.0; type continuous -> revolute

File: robot_quadruped/src/robot_description/urdf/robot.xacro (robot description, xacro)
@@ -264,75 +264,87 @@
   </collision>
 </link>
-<joint name="Revolution 1" type="continuous">
+<joint name="Revolution 1" type="revolute">
   <origin xyz="-0.063124 0.043002 -0.072222" rpy="0 0 0"/>
   <parent link="FL_Brazo_1"/>
   <child link="FL_Antebrazo_1"/>
   <axis xyz="0.134783 0.990599 0.023402"/>
-</joint>
-<joint name="Revolution 2" type="continuous">
+  <limit lower="-1.57" upper="1.57" effort="10.0" velocity="5.0"/>
+</joint>
+<joint name="Revolution 2" type="revolute">
   <origin xyz="-0.00625 0.020813 0.001086" rpy="0 0 0"/>
   <parent link="FL_Hombro_1"/>
   <child link="FL_Brazo_1"/>
   <axis xyz="-0.134783 -0.990599 -0.023402"/>
-</joint>
-<joint name="Revolution 3" type="continuous">
+  <limit lower="-1.57" upper="1.57" effort="10.0" velocity="5.0"/>
+</joint>
+<joint name="Revolution 3" type="revolute">
   <origin xyz="0.182872 -0.091608 0.145512" rpy="0 0 0"/>
   <parent link="base_link"/>
   <child link="FL_Hombro_1"/>
   <axis xyz="-0.990874 0.134786 0.001454"/>
-</joint>
-<joint name="Revolution 4" type="continuous">
+  <limit lower="-1.57" upper="1.57" effort="10.0" velocity="5.0"/>
+</joint>
+<joint name="Revolution 4" type="revolute">
   <origin xyz="-0.068203 0.041505 -0.068376" rpy="0 0 0"/>
   <parent link="RL_Brazo_1"/>
   <child link="RL_Antebrazo_1"/>
   <axis xyz="0.134773 0.990853 -0.006819"/>
-</joint>
-<joint name="Revolution 5" type="continuous">
+  <limit lower="-1.57" upper="1.57" effort="10.0" velocity="5.0"/>
+</joint>
+<joint name="Revolution 5" type="revolute">
   <origin xyz="0.011587 0.01841 0.000462" rpy="0 0 0"/>
   <parent link="RL_Hombro_1"/>
   <child link="RL_Brazo_1"/>
   <axis xyz="0.134773 0.990853 -0.006819"/>
-</joint>
-<joint name="Revolution 6" type="continuous">
+  <limit lower="-1.57" upper="1.57" effort="10.0" velocity="5.0"/>
+</joint>
+<joint name="Revolution 6" type="revolute">
   <origin xyz="-0.027292 -0.06302 0.14582" rpy="0 0 0"/>
   <parent link="base_link"/>
   <child link="RL_Hombro_1"/>
   <axis xyz="-0.990874 0.134786 0.001454"/>
-</joint>
-<joint name="Revolution 7" type="continuous">
+  <limit lower="-1.57" upper="1.57" effort="10.0" velocity="5.0"/>
+</joint>
+<joint name="Revolution 7" type="revolute">
   <origin xyz="-0.079091 -0.012167 -0.068164" rpy="0 0 0"/>
   <parent link="RR_Brazo_1"/>
   <child link="RR_Antebrazo_1"/>
   <axis xyz="0.133564 0.98032 0.145373"/>
-</joint>
-<joint name="Revolution 8" type="continuous">
+  <limit lower="-1.57" upper="1.57" effort="10.0" velocity="5.0"/>
+</joint>
+<joint name="Revolution 8" type="revolute">
   <origin xyz="0.006263 -0.020711 -0.002288" rpy="0 0 0"/>
   <parent link="RR_Hombro_1"/>
   <child link="RR_Brazo_1"/>
   <axis xyz="-0.133564 -0.98032 -0.145373"/>
-</joint>
-<joint name="Revolution 9" type="continuous">
+  <limit lower="-1.57" upper="1.57" effort="10.0" velocity="5.0"/>
+</joint>
+<joint name="Revolution 9" type="revolute">
   <origin xyz="-0.039343 -0.151603 0.145399" rpy="0 0 0"/>
   <parent link="base_link"/>
   <child link="RR_Hombro_1"/>
   <axis xyz="-0.990874 0.134786 0.001454"/>
-</joint>
-<joint name="Revolution 10" type="continuous">
+  <limit lower="-1.57" upper="1.57" effort="10.0" velocity="5.0"/>
+</joint>
+<joint name="Revolution 10" type="revolute">
   <origin xyz="-0.072711 -0.019296 -0.07342" rpy="0 0 0"/>
   <parent link="FR_Brazo_1"/>
   <child link="FR_Antebrazo_1"/>
   <axis xyz="0.134701 0.989734 0.047783"/>
-</joint>
-<joint name="Revolution 11" type="continuous">
+  <limit lower="-1.57" upper="1.57" effort="10.0" velocity="5.0"/>
+</joint>
+<joint name="Revolution 11" type="revolute">
   <origin xyz="-0.015552 -0.017874 -0.000318" rpy="0 0 0"/>
   <parent link="FR_Hombro_1"/>
   <child link="FR_Brazo_1"/>
   <axis xyz="-0.134701 -0.989734 -0.047783"/>
-</joint>
-<joint name="Revolution 12" type="continuous">
+  <limit lower="-1.57" upper="1.57" effort="10.0" velocity="5.0"/>
+</joint>
+<joint name="Revolution 12" type="revolute">
   <origin xyz="0.170768 -0.180587 0.145089" rpy="0 0 0"/>
   <parent link="base_link"/>
   <child link="FR_Hombro_1"/>
   <axis xyz="0.990874 -0.134786 -0.001454"/>
+  <limit lower="-1.57" upper="1.57" effort="10.0" velocity="5.0"/>
 </joint>
 </robot>

Commit message: Adjusted joints positions

File: robot_quadruped/src/robot_description/urdf/robot.urdf (robot description, URDF)
Before this commit: robot robot, 13 links, 12 joints
Links:
- added link imu_link, mass 0.01
- added link world
- link FL_Antebrazo_1: mass 0.011017130901550822 -> 0.11017130901550822; geometry collision mesh filename=file:///home/lucia/TFG/robot_quadruped/src/robot_descriptio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 scale=0.02 0.02 0.02; visual mesh filename=file:///home/lucia/TFG/robot_quadruped/src/robot_descriptio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 scale=0.02 0.02 0.02
- link FL_Brazo_1: mass 0.030409136144975923 -> 0.30409136144975923; geometry collision mesh filename=file:///home/lucia/TFG/robot_quadruped/src/robot_descriptio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 scale=0.02 0.02 0.02; visual mesh filename=file:///home/lucia/TFG/robot_quadruped/src/robot_descriptio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 scale=0.02 0.02 0.02
- link FL_Hombro_1: mass 0.01859774303312477 -> 0.1859774303312477; geometry collision mesh filename=file:///home/lucia/TFG/robot_quadruped/src/robot_descriptio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 scale=0.02 0.02 0.02; visual mesh filename=file:///home/lucia/TFG/robot_quadruped/src/robot_descriptio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 scale=0.02 0.02 0.02
- link FR_Antebrazo_1: mass 0.011033575580722182 -> 0.11033575580722182; geometry collision mesh filename=file:///home/lucia/TFG/robot_quadruped/src/robot_descriptio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 scale=0.02 0.02 0.02; visual mesh filename=file:///home/lucia/TFG/robot_quadruped/src/robot_descriptio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 scale=0.02 0.02 0.02
- link FR_Brazo_1: mass 0.03040973749414956 -> 0.3040973749414956; geometry collision mesh filename=file:///home/lucia/TFG/robot_quadruped/src/robot_descriptio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 scale=0.02 0.02 0.02; visual mesh filename=file:///home/lucia/TFG/robot_quadruped/src/robot_descriptio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 scale=0.02 0.02 0.02
- link FR_Hombro_1: mass 0.01859736994896006 -> 0.1859736994896006; geometry collision mesh filename=file:///home/lucia/TFG/robot_quadruped/src/robot_descriptio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 scale=0.02 0.02 0.02; visual mesh filename=file:///home/lucia/TFG/robot_quadruped/src/robot_descriptio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 scale=0.02 0.02 0.02
- link RL_Antebrazo_1: mass 0.011048026895118968 -> 0.11048026895118968; geometry collision mesh filename=file:///home/lucia/TFG/robot_quadruped/src/robot_descriptio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 scale=0.02 0.02 0.02; visual mesh filename=file:///home/lucia/TFG/robot_quadruped/src/robot_descriptio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 scale=0.02 0.02 0.02
- link RL_Brazo_1: mass 0.03040973749415957 -> 0.3040973749415957; geometry collision mesh filename=file:///home/lucia/TFG/robot_quadruped/src/robot_descriptio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 scale=0.02 0.02 0.02; visual mesh filename=file:///home/lucia/TFG/robot_quadruped/src/robot_descriptio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 scale=0.02 0.02 0.02
- link RL_Hombro_1: mass 0.018594032037447486 -> 0.18594032037447486; geometry collision mesh filename=file:///home/lucia/TFG/robot_quadruped/src/robot_descriptio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 scale=0.02 0.02 0.02; visual mesh filename=file:///home/lucia/TFG/robot_quadruped/src/robot_descriptio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 scale=0.02 0.02 0.02
- link RR_Antebrazo_1: mass 0.011048045171812943 -> 0.11048045171812943; geometry collision mesh filename=file:///home/lucia/TFG/robot_quadruped/src/robot_descriptio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 scale=0.02 0.02 0.02; visual mesh filename=file:///home/lucia/TFG/robot_quadruped/src/robot_descriptio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 scale=0.02 0.02 0.02
- link RR_Brazo_1: mass 0.03040973749415908 -> 0.3040973749415908; geometry collision mesh filename=file:///home/lucia/TFG/robot_quadruped/src/robot_descriptio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 scale=0.02 0.02 0.02; visual mesh filename=file:///home/lucia/TFG/robot_quadruped/src/robot_descriptio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 scale=0.02 0.02 0.02
- link RR_Hombro_1: mass 0.0185940356423774 -> 0.185940356423774; geometry collision mesh filename=file:///home/lucia/TFG/robot_quadruped/src/robot_descriptio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 scale=0.02 0.02 0.02; visual mesh filename=file:///home/lucia/TFG/robot_quadruped/src/robot_descriptio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 scale=0.02 0.02 0.02
- link base_link: geometry collision mesh filename=file:///home/lucia/TFG/robot_quadruped/src/robot_descriptio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 scale=0.02 0.02 0.02; visual mesh filename=file:///home/lucia/TFG/robot_quadruped/src/robot_descriptio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 scale=0.02 0.02 0.02
Joints:
- removed joint Revolution 1
- removed joint Revolution 10
- removed joint Revolution 11
- removed joint Revolution 12
- removed joint Revolution 2
- removed joint Revolution 3
- removed joint Revolution 4
- removed joint Revolution 5
- removed joint Revolution 6
- removed joint Revolution 7
- removed joint Revolution 8
- removed joint Revolution 9
- added joint Revolution_1: type revolute, parent FL_Brazo_1, child FL_Antebrazo_1, origin xyz=-1.258 0.8 -1.435 rpy=0 0 0, axis 0 -1 0, limit lower=-1.57 upper=1.57 effort=10.0 velocity=5.0
- added joint Revolution_10: type revolute, parent FR_Brazo_1, child FR_Antebrazo_1, origin xyz=-1.445 -0.32 -1.48 rpy=0 0 0, axis 0 -1 0, limit lower=-1.57 upper=1.57 effort=10.0 velocity=5.0
- added joint Revolution_11: type revolute, parent FR_Hombro_1, child FR_Brazo_1, origin xyz=-0.27 -0.35 -0.01 rpy=0 0 0, axis 0 -1 0, limit lower=-1.57 upper=1.57 effort=10.0 velocity=5.0
- added joint Revolution_12: type revolute, parent base_link, child FR_Hombro_1, origin xyz=3.41 -3.61 2.90722 rpy=0 0 0, axis 1 0 0, limit lower=-1.57 upper=1.57 effort=10.0 velocity=5.0
- added joint Revolution_2: type revolute, parent FL_Hombro_1, child FL_Brazo_1, origin xyz=-0.1155 0.415 0.025 rpy=0 0 0, axis 0 -1 0, limit lower=-1.57 upper=1.57 effort=10.0 velocity=5.0
- added joint Revolution_3: type revolute, parent base_link, child FL_Hombro_1, origin xyz=3.6001245 -1.83513 2.90722 rpy=0 0 0, axis -1 0 0, limit lower=-1.57 upper=1.57 effort=10.0 velocity=5.0
- added joint Revolution_4: type revolute, parent RL_Brazo_1, child RL_Antebrazo_1, origin xyz=-1.358 0.75 -1.355 rpy=0 0 0, axis 0 -1 0, limit lower=-1.57 upper=1.57 effort=10.0 velocity=5.0
- added joint Revolution_5: type revolute, parent RL_Hombro_1, child RL_Brazo_1, origin xyz=0.285 0.34 0.01 rpy=0 0 0, axis 0 -1 0, limit lower=-1.57 upper=1.57 effort=10.0 velocity=5.0
- added joint Revolution_6: type revolute, parent base_link, child RL_Hombro_1, origin xyz=-0.557292 -1.25513 2.91722 rpy=0 0 0, axis -1 0 0, limit lower=-1.57 upper=1.57 effort=10.0 velocity=5.0
- added joint Revolution_7: type revolute, parent RR_Brazo_1, child RR_Antebrazo_1, origin xyz=-1.59 -0.15 -1.4 rpy=0 0 0, axis 0 -1 0, limit lower=-1.57 upper=1.57 effort=10.0 velocity=5.0
- added joint Revolution_8: type revolute, parent RR_Hombro_1, child RR_Brazo_1, origin xyz=0.18 -0.415 -0.035 rpy=0 0 0, axis 0 -1 0, limit lower=-1.57 upper=1.57 effort=10.0 velocity=5.0
- added joint Revolution_9: type revolute, parent base_link, child RR_Hombro_1, origin xyz=-0.8 -3.03 2.9 rpy=0 0 0, axis 1 0 0, limit lower=-1.57 upper=1.57 effort=10.0 velocity=5.0
- added joint fixed_base_joint: type fixed, parent world, child base_link, origin xyz=0 0 2.35 rpy=0 0 0
- added joint imu_joint: type fixed, parent base_link, child imu_link

Commit message: Control not working because of bridge

File: robot_quadruped/src/robot_description/urdf/robot.urdf (robot description, URDF)
Before this commit: robot robot, 15 links, 14 joints
Links:
- removed link FL_Antebrazo_1
- removed link FL_Brazo_1
- removed link FL_Hombro_1
- removed link FR_Antebrazo_1
- removed link FR_Brazo_1
- removed link FR_Hombro_1
- removed link RL_Antebrazo_1
- removed link RL_Brazo_1
- removed link RL_Hombro_1
- removed link RR_Antebrazo_1
- removed link RR_Brazo_1
- removed link RR_Hombro_1
- added link FL_Antebrazo, mass 0.11017130901550822; collision mesh filename=file:///home/lucia/TFG/robot_quadruped/src/robot_descriptio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 scale=0.02 0.02 0.02; visual mesh filename=file:///home/lucia/TFG/robot_quadruped/src/robot_descriptio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 scale=0.02 0.02 0.02
- added link FL_Brazo, mass 0.30409136144975923; collision mesh filename=file:///home/lucia/TFG/robot_quadruped/src/robot_descriptio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 scale=0.02 0.02 0.02; visual mesh filename=file:///home/lucia/TFG/robot_quadruped/src/robot_descriptio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 scale=0.02 0.02 0.02
- added link FL_Hombro, mass 0.1859774303312477; collision mesh filename=file:///home/lucia/TFG/robot_quadruped/src/robot_descriptio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 scale=0.02 0.02 0.02; visual mesh filename=file:///home/lucia/TFG/robot_quadruped/src/robot_descriptio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 scale=0.02 0.02 0.02
- added link FR_Antebrazo, mass 0.11033575580722182; collision mesh filename=file:///home/lucia/TFG/robot_quadruped/src/robot_descriptio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 scale=0.02 0.02 0.02; visual mesh filename=file:///home/lucia/TFG/robot_quadruped/src/robot_descriptio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 scale=0.02 0.02 0.02
- added link FR_Brazo, mass 0.3040973749414956; collision mesh filename=file:///home/lucia/TFG/robot_quadruped/src/robot_descriptio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 scale=0.02 0.02 0.02; visual mesh filename=file:///home/lucia/TFG/robot_quadruped/src/robot_descriptio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 scale=0.02 0.02 0.02
- added link FR_Hombro, mass 0.1859736994896006; collision mesh filename=file:///home/lucia/TFG/robot_quadruped/src/robot_descriptio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 scale=0.02 0.02 0.02; visual mesh filename=file:///home/lucia/TFG/robot_quadruped/src/robot_descriptio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 scale=0.02 0.02 0.02
- added link RL_Antebrazo, mass 0.11048026895118968; collision mesh filename=file:///home/lucia/TFG/robot_quadruped/src/robot_descriptio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 scale=0.02 0.02 0.02; visual mesh filename=file:///home/lucia/TFG/robot_quadruped/src/robot_descriptio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 scale=0.02 0.02 0.02
- added link RL_Brazo, mass 0.3040973749415957; collision mesh filename=file:///home/lucia/TFG/robot_quadruped/src/robot_descriptio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 scale=0.02 0.02 0.02; visual mesh filename=file:///home/lucia/TFG/robot_quadruped/src/robot_descriptio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 scale=0.02 0.02 0.02
- added link RL_Hombro, mass 0.18594032037447486; collision mesh filename=file:///home/lucia/TFG/robot_quadruped/src/robot_descriptio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 scale=0.02 0.02 0.02; visual mesh filename=file:///home/lucia/TFG/robot_quadruped/src/robot_descriptio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 scale=0.02 0.02 0.02
- added link RR_Antebrazo, mass 0.11048045171812943; collision mesh filename=file:///home/lucia/TFG/robot_quadruped/src/robot_descriptio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 scale=0.02 0.02 0.02; visual mesh filename=file:///home/lucia/TFG/robot_quadruped/src/robot_descriptio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 scale=0.02 0.02 0.02
- added link RR_Brazo, mass 0.3040973749415908; collision mesh filename=file:///home/lucia/TFG/robot_quadruped/src/robot_descriptio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 scale=0.02 0.02 0.02; visual mesh filename=file:///home/lucia/TFG/robot_quadruped/src/robot_descriptio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 scale=0.02 0.02 0.02
- added link RR_Hombro, mass 0.185940356423774; collision mesh filename=file:///home/lucia/TFG/robot_quadruped/src/robot_descriptio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 scale=0.02 0.02 0.02; visual mesh filename=file:///home/lucia/TFG/robot_quadruped/src/robot_descriptio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 scale=0.02 0.02 0.02
- link imu_link: mass 0.01 -> 0.5
Joints:
- joint Revolution_1: child FL_Antebrazo_1 -> FL_Antebrazo; parent FL_Brazo_1 -> FL_Brazo
- joint Revolution_10: child FR_Antebrazo_1 -> FR_Antebrazo; parent FR_Brazo_1 -> FR_Brazo
- joint Revolution_11: child FR_Brazo_1 -> FR_Brazo; parent FR_Hombro_1 -> FR_Hombro
- joint Revolution_12: child FR_Hombro_1 -> FR_Hombro
- joint Revolution_2: child FL_Brazo_1 -> FL_Brazo; parent FL_Hombro_1 -> FL_Hombro
- joint Revolution_3: child FL_Hombro_1 -> FL_Hombro
- joint Revolution_4: child RL_Antebrazo_1 -> RL_Antebrazo; parent RL_Brazo_1 -> RL_Brazo
- joint Revolution_5: child RL_Brazo_1 -> RL_Brazo; parent RL_Hombro_1 -> RL_Hombro
- joint Revolution_6: child RL_Hombro_1 -> RL_Hombro
- joint Revolution_7: child RR_Antebrazo_1 -> RR_Antebrazo; parent RR_Brazo_1 -> RR_Brazo
- joint Revolution_8: child RR_Brazo_1 -> RR_Brazo; parent RR_Hombro_1 -> RR_Hombro
- joint Revolution_9: child RR_Hombro_1 -> RR_Hombro

Commit message: funshiona

File: robot_quadruped/src/robot_description/urdf/robot.urdf (robot description, URDF)
Before this commit: robot robot, 15 links, 14 joints
Links:
- link imu_link: mass 0.01 -> 0.1
